File: pwm_pcb/pwm_pcb.kicad_sch (KiCad schematic)
At the start: 69 parts, among them J1 Conn_01x02, J2 Conn_01x02, J3 Conn_01x16, Q1 NMOS, Q10 NMOS, Q11 NMOS, Q12 NMOS, Q13 NMOS, Q14 NMOS, Q15 NMOS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

Commit message: adding test code and 3d print files
Other:
- note added: "when VDC is applied (8-37V), and the 5v is shorted to ground, the fuse doesnt pop, D3 gets blown out"
Changed lines of the file:
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@@
     (stroke (width 0) (type default) (color 0 0 0 0))
+  )
+  (text "when VDC is applied (8-37V), and the 5v \nis shorted to ground, the fuse doesnt pop,\nD3 gets blown out\n"
+    (at 224.79 7.62 0)
+    (effects (font (size 1.27 1.27)) (justify left bottom))
   )
   (text "5V only in!" (at 247.65 95.25 0)
