File: pwm_pcb_larger/pwm_pcb_larger.kicad_sch (KiCad schematic)
At the start: 84 parts, among them J1 Conn_01x02, J10 Conn_01x02, J11 Conn_01x02, J12 Conn_01x02, J13 Conn_01x02, J14 Conn_01x02, J15 Conn_01x02, J16 Conn_01x02, J17 Conn_01x02, J18 Conn_01x02, J2 Conn_01x02, J3 Conn_01x02, J4 Conn_01x02, J5 Conn_01x02, J6 Conn_01x02, J7 Conn_01x02, J8 Conn_01x02, J9 Conn_01x02, Q1 NMOS, Q10 NMOS, Q11 NMOS, Q12 NMOS, Q13 NMOS, Q14 NMOS, Q15 NMOS, Q16 NMOS, Q17 Q_PMOS_DGS, Q2 NMOS, Q3 NMOS, Q4 NMOS, Q5 NMOS, Q6 NMOS, Q7 NMOS, Q8 NMOS, Q9 NMOS, SW1 SW_SPST, U1 ESP32_DevKit_V1_DOIT, U2 LM317_TO-252

Commit message: updating the new rev board with new connectors for led outputs and PSU input
Parts:
- added H1, H2, H3, H4: MountingHole, MountingHole:MountingHole_3.2mm_M3, symbol Mechanical:MountingHole
- J1, J2: footprint Connector_Phoenix_MSTB:PhoenixContact_MSTBVA_2,5_2-G-5,08_1x02_P5.08mm_Vertical -> william customs:Kobiconn - 2 pin terminal - 158P02DT39BE
- J10, J11, J12, J13, J14, J15, J16, J17, J18, J3, J4, J5, J6, J7, J8, J9: footprint Connector_Molex:Molex_Micro-Fit_3.0_43650-0200_1x02_P3.00mm_Horizontal -> Connector_Molex:Molex_Micro-Fit_3.0_43045-0212_2x01_P3.00mm_Vertical

Commit message: rev 3 finished and sent to JLC for fab
Parts:
- D1, D2: footprint LED_SMD:LED_1206_3216Metric -> LED_SMD:LED_0805_2012Metric
- Q17: symbol Device:Q_PMOS_DGS -> Device:Q_PMOS_GSD
Connections:
- net esp32_power: now also Q17.1 (G); no longer Q17.2 (G)
- net at F1.1, SW1.2 (B): now also Q17.2 (S); no longer Q17.3 (S)
- net at D1.2 (A): now also Q17.3 (D); no longer Q17.1 (D)
Other:
- note added: "Drain"
- note added: "Gate"
- note added: "Source"
Changed lines of the file:
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@@
 		)
 	)
+	(text "Source"
+		(exclude_from_sim no)
+		(at 162.306 37.084 0)
+		(effects
+			(font
+				(size 1.27 1.27)
+			)
+		)
+	)
+	(text "Drain\n	\n"
+		(exclude_from_sim no)
+		(at 164.084 47.498 0)
+		(effects
+			(font
+				(size 1.27 1.27)
+			)
+		)
+	)
 	(text "8V - 37V	"
 		(exclude_from_sim no)
@@
 		)
 	)
+	(text "Gate"
+		(exclude_from_sim no)
+		(at 174.752 39.116 0)
+		(effects
+			(font
+				(size 1.27 1.27)
+			)
+		)
+	)
 	(text "protection circuitry"
 		(exclude_from_sim no)
@@
 			)
 		)
-		(property "Footprint" "LED_SMD:LED_1206_3216Metric"
+		(property "Footprint" "LED_SMD:LED_0805_2012Metric"
 			(at 189.23 43.18 0)
 			(effects
@@
 	)
 	(symbol
-		(lib_id "Device:Q_PMOS_DGS")
+		(lib_id "Device:Q_PMOS_GSD")
 		(at 171.45 41.91 180)
 		(unit 1)
@@
 			)
 		)
-		(property "Description" ""
+		(property "Description" "P-MOSFET transistor, gate/source/drain"
 			(at 171.45 41.91 0)
 			(effects
@@
 			)
 		)
-		(property "Footprint" "LED_SMD:LED_1206_3216Metric"
+		(property "Footprint" "LED_SMD:LED_0805_2012Metric"
 			(at 168.91 50.8 0)
 			(effects
